File: design files/board.kicad_pcb (KiCad board)
At the start: 2 copper layers, 40 x 30 mm, 40 parts, among them J1 USB_C_Receptacle_PowerOnly_6P, J3 Conn_01x02_Pin, Q1 Q_PMOS_GDS, U1 TPS61089, U2 BQ25306RTER

Commit message: updated design
Parts:
- D2: footprint Diode_SMD:D_1206_3216Metric -> Diode_SMD:D_SMA
- moved D2 0.61 mm to (28.9, 14.4)
Routing:
- net VBUS: track 48.5 -> 48.6 mm, vias 7 -> 10
