File: design files/board.kicad_sch (KiCad schematic)
At the start: 40 parts, among them J1 USB_C_Receptacle_PowerOnly_6P, J3 Conn_01x02_Pin, Q1 Q_PMOS_GDS, U1 TPS61089, U2 BQ25306RTER

Commit message: updated design
Parts:
- D2: footprint Diode_SMD:D_1206_3216Metric -> Diode_SMD:D_SMA
Changed lines of the file:
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@@
 			)
 		)
-		(property "Footprint" "Diode_SMD:D_1206_3216Metric"
+		(property "Footprint" "Diode_SMD:D_SMA"
 			(at 238.76 35.56 0)
 			(hide yes)
